Commit message: fix lenght values

File: src/three_finger_hand/urdf/three_finger_hand.urdf.xacro (robot description, xacro)
@@ -30,11 +30,11 @@
   </link>
   <xacro:finger prefix="finger_1" parent="palm">
-    <origin xyz="0.05 0 0.08" rpy="0 0.52333333 0"/><!-- <origin xyz="0.06785 -0.002 0.08" rpy="0 0.52333333 0"/> -->
+    <origin xyz="0.05785 0 0.06375" rpy="0 0.52333333 0"/>
   </xacro:finger>
   <xacro:finger prefix="finger_2" parent="palm">
-    <origin xyz="-0.025 0.043 0.08" rpy="0 0.52333333 2.0944"/>
+    <origin xyz="-0.02893 0.05001 0.06375" rpy="0 0.52333333 2.0944"/>
   </xacro:finger>
   <xacro:finger prefix="finger_3" parent="palm">
-    <origin xyz="-0.025 -0.043 0.08" rpy="0 0.52333333 -2.0944"/>
+    <origin xyz="-0.02893 -0.05001 0.06375" rpy="0 0.52333333 -2.0944"/>
   </xacro:finger>
 </robot>

Commit message: add files related gazebo sim

File: src/three_finger_hand/urdf/three_finger_hand.urdf.xacro (robot description, xacro)
@@ -38,3 +38,74 @@
     <origin xyz="-0.02893 -0.05001 0.06375" rpy="0 0.52333333 -2.0944"/>
   </xacro:finger>
+  <gazebo>
+    <plugin filename="libgz_ros2_control-system.so"
+            name="gz_ros2_control::GazeboSimROS2ControlPlugin">
+      <parameters>$(find three_finger_hand)/config/hand_controller.yaml</parameters>
+    </plugin>
+  </gazebo>
+  <ros2_control name="GazeboSystem" type="system">
+    <hardware>
+      <plugin>gz_ros2_control/GazeboSimSystem</plugin>
+    </hardware>
+    <joint name="finger_1_joint_1">
+      <command_interface name="position"><param name="min">-1.57</param><param name="max">1.57</param></command_interface>
+      <state_interface name="position"/>
+      <state_interface name="velocity"/>
+    </joint>
+    <joint name="finger_1_joint_2">
+      <command_interface name="position"><param name="min">0.0</param><param name="max">1.57</param></command_interface>
+      <state_interface name="position"/>
+      <state_interface name="velocity"/>
+    </joint>
+    <joint name="finger_1_joint_3">
+      <command_interface name="position"><param name="min">0.0</param><param name="max">1.57</param></command_interface>
+      <state_interface name="position"/>
+      <state_interface name="velocity"/>
+    </joint>
+    <joint name="finger_1_joint_4">
+      <command_interface name="position"><param name="min">0.0</param><param name="max">1.57</param></command_interface>
+      <state_interface name="position"/>
+      <state_interface name="velocity"/>
+    </joint>
+    <joint name="finger_2_joint_1">
+      <command_interface name="position"><param name="min">-1.57</param><param name="max">1.57</param></command_interface>
+      <state_interface name="position"/>
+      <state_interface name="velocity"/>
+    </joint>
+    <joint name="finger_2_joint_2">
+      <command_interface name="position"><param name="min">0.0</param><param name="max">1.57</param></command_interface>
+      <state_interface name="position"/>
+      <state_interface name="velocity"/>
+    </joint>
+    <joint name="finger_2_joint_3">
+      <command_interface name="position"><param name="min">0.0</param><param name="max">1.57</param></command_interface>
+      <state_interface name="position"/>
+      <state_interface name="velocity"/>
+    </joint>
+    <joint name="finger_2_joint_4">
+      <command_interface name="position"><param name="min">0.0</param><param name="max">1.57</param></command_interface>
+      <state_interface name="position"/>
+      <state_interface name="velocity"/>
+    </joint>
+    <joint name="finger_3_joint_1">
+      <command_interface name="position"><param name="min">-1.57</param><param name="max">1.57</param></command_interface>
+      <state_interface name="position"/>
+      <state_interface name="velocity"/>
+    </joint>
+    <joint name="finger_3_joint_2">
+      <command_interface name="position"><param name="min">0.0</param><param name="max">1.57</param></command_interface>
+      <state_interface name="position"/>
+      <state_interface name="velocity"/>
+    </joint>
+    <joint name="finger_3_joint_3">
+      <command_interface name="position"><param name="min">0.0</param><param name="max">1.57</param></command_interface>
+      <state_interface name="position"/>
+      <state_interface name="velocity"/>
+    </joint>
+    <joint name="finger_3_joint_4">
+      <command_interface name="position"><param name="min">0.0</param><param name="max">1.57</param></command_interface>
+      <state_interface name="position"/>
+      <state_interface name="velocity"/>
+    </joint>
+  </ros2_control>
 </robot>

Commit message: add functionality of ik for circular motion

File: src/three_finger_hand/urdf/three_finger_hand.urdf.xacro (robot description, xacro)
@@ -30,5 +30,5 @@
   </link>
   <xacro:finger prefix="finger_1" parent="palm">
-    <origin xyz="0.05785 0 0.06375" rpy="0 0.52333333 0"/>
+    <origin xyz="0.05777 0 0.06375" rpy="0 0.52333333 0"/>
   </xacro:finger>
   <xacro:finger prefix="finger_2" parent="palm">
