Commit message: minor fixes

File: src/three_finger_hand/urdf/finger.xacro (robot description, xacro)
@@ -6,5 +6,5 @@
       <child link="${prefix}_knuckle"/>
       <xacro:insert_block name="origin"/>
-      <axis xyz="0 1 0"/> <limit lower="-1.57" upper="1.57" effort="10" velocity="1.0"/>
+      <axis xyz="1 0 0"/> <limit lower="-1.57" upper="1.57" effort="10" velocity="1.0"/>
     </joint>
     <link name="${prefix}_knuckle">
@@ -32,6 +32,6 @@
       <parent link="${prefix}_knuckle"/>
       <child link="${prefix}_proximal"/>
-      <origin xyz="0 0 0.01025" rpy="0 0 0"/>
-      <axis xyz="1 0 0"/> <limit lower="0.0" upper="1.57" effort="10" velocity="1.0"/>
+      <origin xyz="0 0 0.07" rpy="0 0 1.57"/>
+      <axis xyz="1 0 0"/> <limit lower="-1.57" upper="1.57" effort="10" velocity="1.0"/>
     </joint>
     <link name="${prefix}_proximal">
@@ -57,7 +57,7 @@
       <parent link="${prefix}_proximal"/>
       <child link="${prefix}_middle"/>
-      <origin xyz="0 0 0.07" rpy="0 0 0"/>
-      <axis xyz="1 0 0"/>
-      <limit lower="0.0" upper="1.57" effort="10" velocity="1.0"/>
+      <origin xyz="0 0 0.01025" rpy="0 0 -1.57"/>
+      <axis xyz="0 1 0"/>
+      <limit lower="-1.57" upper="1.57" effort="10" velocity="1.0"/>
     </joint>
     <link name="${prefix}_middle">
@@ -84,6 +84,6 @@
       <child link="${prefix}_distal"/>
       <origin xyz="0 0 0.07" rpy="0 0 0"/>
-      <axis xyz="1 0 0"/>
-      <limit lower="0.0" upper="1.57" effort="10" velocity="1.0"/>
+      <axis xyz="0 1 0"/>
+      <limit lower="-1.57" upper="1.57" effort="10" velocity="1.0"/>
     </joint>
     <link name="${prefix}_distal">

File: src/three_finger_hand/urdf/three_finger_hand.urdf.xacro (robot description, xacro)
@@ -6,9 +6,9 @@
     <parent link="world"/>
     <child link="palm"/>
-    <origin xyz="0 0 0.1" rpy="0 0 0"/>
+    <origin xyz="0 0 0" rpy="0 0 0"/>
   </joint>
   <link name="palm">
     <visual>
-      <origin xyz="0 0 0" rpy="0 0 0"/>
+      <origin xyz="0 0 0" rpy="0 0 0.523"/>
       <geometry>
         <mesh filename="package://three_finger_hand/meshes/palm.stl" scale="0.001 0.001 0.001"/>
@@ -30,11 +30,11 @@
   </link>
   <xacro:finger prefix="finger_1" parent="palm">
-    <origin xyz="0.05 0 0.02" rpy="0 0 0"/>
+    <origin xyz="0.05 0 0.08" rpy="0 0.52333333 0"/><!-- <origin xyz="0.06785 -0.002 0.08" rpy="0 0.52333333 0"/> -->
   </xacro:finger>
   <xacro:finger prefix="finger_2" parent="palm">
-    <origin xyz="-0.025 0.043 0.02" rpy="0 0 2.0944"/>
+    <origin xyz="-0.025 0.043 0.08" rpy="0 0.52333333 2.0944"/>
   </xacro:finger>
   <xacro:finger prefix="finger_3" parent="palm">
-    <origin xyz="-0.025 -0.043 0.02" rpy="0 0 -2.0944"/>
+    <origin xyz="-0.025 -0.043 0.08" rpy="0 0.52333333 -2.0944"/>
   </xacro:finger>
 </robot>

Commit message: Add CLI support for circle waypoint generation and enhance GUI for finger positioning

File: src/three_finger_hand/urdf/finger.xacro (robot description, xacro)
@@ -35,5 +35,5 @@
       <child link="${prefix}_proximal"/>
       <origin xyz="0 0 0.01025" rpy="0 0 1.57"/>
-      <axis xyz="1 0 0"/> <limit lower="-0.628" upper="1.256" effort="10" velocity="1.0"/>
+      <axis xyz="1 0 0"/> <limit lower="-1.256" upper="1.256" effort="10" velocity="1.0"/>
       <damping value="0.5"/>
       <dynamics friction="0.5"/>

File: src/three_finger_hand/urdf/three_finger_hand.urdf.xacro (robot description, xacro)
@@ -58,5 +58,5 @@
     <joint name="finger_1_joint_2">
       <command_interface name="position">
-        <param name="min">-0.628</param>
+        <param name="min">-1.256</param>
         <param name="max">1.256</param>
       </command_interface>
@@ -90,5 +90,5 @@
     <joint name="finger_2_joint_2">
       <command_interface name="position">
-        <param name="min">-0.628</param>
+        <param name="min">-1.256</param>
         <param name="max">1.256</param>
       </command_interface>
@@ -122,5 +122,5 @@
     <joint name="finger_3_joint_2">
       <command_interface name="position">
-        <param name="min">-0.628</param>
+        <param name="min">-1.256</param>
         <param name="max">1.256</param>
       </command_interface>
